File: SmartishFairy.kicad_sch (KiCad schematic)
At the start: 14 parts, among them J1 USB_C_Receptacle_USB2.0, J10 Conn_01x02_Pin, J13 Data_In, J14 Data_Out, J3 Screw_Terminal_01x02, J4 Screw_Terminal_01x02, J5 Screw_Terminal_01x02, J6 Screw_Terminal_01x06, J7 Screw_Terminal_01x06, J8 Screw_Terminal_01x06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

Commit message: ECR fixes
Parts:
- added J15: Ctl_Pwr, symbol Connector:Screw_Terminal_01x02
- J3: value Screw_Terminal_01x02 -> IN1
- J4: value Screw_Terminal_01x02 -> IN2
- J5: value Screw_Terminal_01x02 -> IN3
- J6: value Screw_Terminal_01x06 -> OUT1
- J7: value Screw_Terminal_01x06 -> OUT2
- J8: value Screw_Terminal_01x06 -> OUT3
Connections:
- net GND: now also U4.8 (OE), J15.2 (Pin_2)
- net VBUS: now also J15.1 (Pin_1)
Other:
- sheet Controller ports: added +3V3; removed 3V3
Changed lines of the file:
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@@
   (junction (at 224.79 29.21) (diameter 0) (color 0 0 0 0)
   )
+  (junction (at 60.96 24.13) (diameter 0) (color 0 0 0 0)
+  )
   (junction (at 224.79 74.93) (diameter 0) (color 0 0 0 0)
   )
@@
   )
   (junction (at 54.61 102.87) (diameter 0) (color 0 0 0 0)
+  )
+  (junction (at 91.44 26.67) (diameter 0) (color 0 0 0 0)
+  )
+  (junction (at 91.44 24.13) (diameter 0) (color 0 0 0 0)
   )
   (no_connect (at 69.85 170.18))
@@
     (stroke (width 0) (type default))
   )
+  (wire (pts (xy 102.87 152.4) (xy 102.87 149.86))
+    (stroke (width 0) (type default))
+  )
   (wire (pts (xy 35.56 154.94) (xy 38.1 154.94))
     (stroke (width 0) (type default))
@@
     (stroke (width 0) (type default))
   )
+  (wire (pts (xy 93.98 24.13) (xy 91.44 24.13))
+    (stroke (width 0) (type default))
+  )
   (wire (pts (xy 66.04 105.41) (xy 66.04 107.95))
     (stroke (width 0) (type default))
@@
     (stroke (width 0) (type default))
   )
+  (wire (pts (xy 102.87 149.86) (xy 90.17 149.86))
+    (stroke (width 0) (type default))
+  )
   (wire (pts (xy 53.34 107.95) (xy 54.61 107.95))
     (stroke (width 0) (type default))
@@
     (stroke (width 0) (type default))
   )
+  (wire (pts (xy 91.44 24.13) (xy 91.44 21.59))
+    (stroke (width 0) (type default))
+  )
   (wire (pts (xy 104.14 113.03) (xy 109.22 113.03))
     (stroke (width 0) (type default))
@@
     (stroke (width 0) (type default))
   )
+  (wire (pts (xy 91.44 26.67) (xy 91.44 29.21))
+    (stroke (width 0) (type default))
+  )
   (wire (pts (xy 224.79 119.38) (xy 224.79 121.92))
     (stroke (width 0) (type default))
   )
   (wire (pts (xy 224.79 46.99) (xy 224.79 52.07))
+    (stroke (width 0) (type default))
+  )
+  (wire (pts (xy 93.98 26.67) (xy 91.44 26.67))
     (stroke (width 0) (type default))
   )
@@
       (effects (font (size 1.27 1.27)) (justify left))
     )
-    (property "Value" "Screw_Terminal_01x02" (at 71.12 27.305 0)
+    (property "Value" "IN1" (at 71.12 27.305 0)
       (effects (font (size 1.27 1.27)) (justify left))
     )
@@
         (path "/c494d399-9c3e-4fb0-8fd0-96c74769e433"
           (reference "J3") (unit 1)
+        )
+      )
+    )
+  )
+  (symbol (lib_id "power:PWR_FLAG") (at 60.96 24.13 90) (unit 1)
+    (in_bom yes) (on_board yes) (dnp no) (fields_autoplaced)
+    (property "Reference" "#FLG01" (at 59.055 24.13 0)
+      (effects (font (size 1.27 1.27)) hide)
+    )
+    (property "Value" "PWR_FLAG" (at 57.15 24.765 90)
+      (effects (font (size 1.27 1.27)) (justify left))
+    )
+    (property "Footprint" "" (at 60.96 24.13 0)
+      (effects (font (size 1.27 1.27)) hide)
+    )
+    (property "Datasheet" "~" (at 60.96 24.13 0)
+      (effects (font (size 1.27 1.27)) hide)
+    )
+    (pin "1")
+    (instances
+      (project "SmartishFairy"
+        (path "/c494d399-9c3e-4fb0-8fd0-96c74769e433"
+          (reference "#FLG01") (unit 1)
         )
       )
@@
       (effects (font (size 1.27 1.27)) (justify left))
     )
-    (property "Value" "Screw_Terminal_01x06" (at 236.22 88.265 0)
+    (property "Value" "OUT2" (at 236.22 88.265 0)
       (effects (font (size 1.27 1.27)) (justify left))
     )
@@
       (effects (font (size 1.27 1.27)) (justify left))
     )
-    (property "Value" "Screw_Terminal_01x02" (at 71.12 47.625 0)
+    (property "Value" "IN2" (at 71.12 47.625 0)
       (effects (font (size 1.27 1.27)) (justify left))
     )
@@
         (path "/c494d399-9c3e-4fb0-8fd0-96c74769e433"
           (reference "J4") (unit 1)
+        )
+      )
+    )
+  )
+  (symbol (lib_id "power:GND") (at 102.87 152.4 0) (unit 1)
+    (in_bom yes) (on_board yes) (dnp no) (fields_autoplaced)
+    (property "Reference" "#PWR091" (at 102.87 158.75 0)
+      (effects (font (size 1.27 1.27)) hide)
+    )
+    (property "Value" "GND" (at 102.87 157.48 0)
+      (effects (font (size 1.27 1.27)))
+    )
+    (property "Footprint" "" (at 102.87 152.4 0)
+      (effects (font (size 1.27 1.27)) hide)
+    )
+    (property "Datasheet" "" (at 102.87 152.4 0)
+      (effects (font (size 1.27 1.27)) hide)
+    )
+    (pin "1")
+    (instances
+      (project "SmartishFairy"
+        (path "/c494d399-9c3e-4fb0-8fd0-96c74769e433"
+          (reference "#PWR091") (unit 1)
         )
       )
@@
     )
   )
+  (symbol (lib_id "power:PWR_FLAG") (at 91.44 24.13 90) (unit 1)
+    (in_bom yes) (on_board yes) (dnp no) (fields_autoplaced)
+    (property "Reference" "#FLG02" (at 89.535 24.13 0)
+      (effects (font (size 1.27 1.27)) hide)
+    )
+    (property "Value" "PWR_FLAG" (at 87.63 24.765 90)
+      (effects (font (size 1.27 1.27)) (justify left))
+    )
+    (property "Footprint" "" (at 91.44 24.13 0)
+      (effects (font (size 1.27 1.27)) hide)
+    )
+    (property "Datasheet" "~" (at 91.44 24.13 0)
+      (effects (font (size 1.27 1.27)) hide)
+    )
+    (pin "1")
+    (instances
+      (project "SmartishFairy"
+        (path "/c494d399-9c3e-4fb0-8fd0-96c74769e433"
+          (reference "#FLG02") (unit 1)
+        )
+      )
+    )
+  )
+  (symbol (lib_id "power:PWR_FLAG") (at 91.44 26.67 90) (unit 1)
+    (in_bom yes) (on_board yes) (dnp no) (fields_autoplaced)
+    (property "Reference" "#FLG03" (at 89.535 26.67 0)
+      (effects (font (size 1.27 1.27)) hide)
+    )
+    (property "Value" "PWR_FLAG" (at 87.63 27.305 90)
+      (effects (font (size 1.27 1.27)) (justify left))
+    )
+    (property "Footprint" "" (at 91.44 26.67 0)
+      (effects (font (size 1.27 1.27)) hide)
+    )
+    (property "Datasheet" "~" (at 91.44 26.67 0)
+      (effects (font (size 1.27 1.27)) hide)
+    )
+    (pin "1")
+    (instances
+      (project "SmartishFairy"
+        (path "/c494d399-9c3e-4fb0-8fd0-96c74769e433"
+          (reference "#FLG03") (unit 1)
+        )
+      )
+    )
+  )
   (symbol (lib_id "Connector:Screw_Terminal_01x06") (at 233.68 39.37 0) (unit 1)
     (in_bom yes) (on_board yes) (dnp no) (fields_autoplaced)
@@
       (effects (font (size 1.27 1.27)) (justify left))
     )
-    (property "Value" "Screw_Terminal_01x06" (at 236.22 42.545 0)
+    (property "Value" "OUT1" (at 236.22 42.545 0)
       (effects (font (size 1.27 1.27)) (justify left))
     )
@@
     )
   )
+  (symbol (lib_id "power:VBUS") (at 91.44 21.59 0) (unit 1)
+    (in_bom yes) (on_board yes) (dnp no) (fields_autoplaced)
+    (property "Reference" "#PWR089" (at 91.44 25.4 0)
+      (effects (font (size 1.27 1.27)) hide)
+    )
+    (property "Value" "VBUS" (at 91.44 17.78 0)
+      (effects (font (size 1.27 1.27)))
+    )
+    (property "Footprint" "" (at 91.44 21.59 0)
+      (effects (font (size 1.27 1.27)) hide)
+    )
+    (property "Datasheet" "" (at 91.44 21.59 0)
+      (effects (font (size 1.27 1.27)) hide)
+    )
+    (pin "1")
+    (instances
+      (project "SmartishFairy"
+        (path "/c494d399-9c3e-4fb0-8fd0-96c74769e433"
+          (reference "#PWR089") (unit 1)
+        )
+      )
+    )
+  )
   (symbol (lib_id "power:GND") (at 60.96 49.53 0) (unit 1)
     (in_bom yes) (on_board yes) (dnp no) (fields_autoplaced)
@@
     )
   )
+  (symbol (lib_id "power:GND") (at 91.44 29.21 0) (unit 1)
+    (in_bom yes) (on_board yes) (dnp no) (fields_autoplaced)
+    (property "Reference" "#PWR090" (at 91.44 35.56 0)
+      (effects (font (size 1.27 1.27)) hide)
+    )
+    (property "Value" "GND" (at 91.44 34.29 0)
+      (effects (font (size 1.27 1.27)))
+    )
+    (property "Footprint" "" (at 91.44 29.21 0)
+      (effects (font (size 1.27 1.27)) hide)
+    )
+    (property "Datasheet" "" (at 91.44 29.21 0)
+      (effects (font (size 1.27 1.27)) hide)
+    )
+    (pin "1")
+    (instances
+      (project "SmartishFairy"
+        (path "/c494d399-9c3e-4fb0-8fd0-96c74769e433"
+          (reference "#PWR090") (unit 1)
+        )
+      )
+    )
+  )
   (symbol (lib_id "power:VBUS") (at 129.54 49.53 0) (unit 1)
     (in_bom yes) (on_board yes) (dnp no) (fields_autoplaced)
@@
       (effects (font (size 1.27 1.27)) (justify left))
     )
-    (property "Value" "Screw_Terminal_01x06" (at 236.22 135.255 0)
+    (property "Value" "OUT3" (at 236.22 135.255 0)
       (effects (font (size 1.27 1.27)) (justify left))
     )
@@
       (effects (font (size 1.27 1.27)) (justify left))
     )
-    (property "Value" "Screw_Terminal_01x02" (at 71.12 67.945 0)
+    (property "Value" "IN3" (at 71.12 67.945 0)
       (effects (font (size 1.27 1.27)) (justify left))
     )
@@
         (path "/c494d399-9c3e-4fb0-8fd0-96c74769e433"
           (reference "J9") (unit 1)
+        )
+      )
+    )
+  )
+  (symbol (lib_id "Connector:Screw_Terminal_01x02") (at 99.06 24.13 0) (unit 1)
+    (in_bom yes) (on_board yes) (dnp no) (fields_autoplaced)
+    (property "Reference" "J15" (at 101.6 24.765 0)
+      (effects (font (size 1.27 1.27)) (justify left))
+    )
+    (property "Value" "Ctl_Pwr" (at 101.6 27.305 0)
+      (effects (font (size 1.27 1.27)) (justify left))
+    )
+    (property "Footprint" "" (at 99.06 24.13 0)
+      (effects (font (size 1.27 1.27)) hide)
+    )
+    (property "Datasheet" "~" (at 99.06 24.13 0)
+      (effects (font (size 1.27 1.27)) hide)
+    )
+    (pin "1")
+    (pin "2")
+    (instances
+      (project "SmartishFairy"
+        (path "/c494d399-9c3e-4fb0-8fd0-96c74769e433"
+          (reference "J15") (unit 1)
         )
       )
@@
       (effects (font (size 1.27 1.27)) (justify right))
     )
-    (pin "3V3" input (at 135.89 53.34 90)
-      (effects (font (size 1.27 1.27)) (justify right))
-    )
+    (pin "+3V3" output (at 135.89 53.34 90)
+      (effects (font (size 1.27 1.27)) (justify right))
+    )

Commit message: ECR fixes
Parts:
- J10, J9: footprint (none) -> Connector_PinHeader_2.54mm:PinHeader_1x02_P2.54mm_Vertical
- J13, J14: footprint (none) -> TerminalBlock_TE-Connectivity:TerminalBlock_TE_282834-4_1x04_P2.54mm_Horizontal
- J15, J3, J4, J5: footprint (none) -> TerminalBlock_TE-Connectivity:TerminalBlock_TE_282834-2_1x02_P2.54mm_Horizontal
- J6, J7, J8: footprint (none) -> TerminalBlock_TE-Connectivity:TerminalBlock_TE_282834-6_1x06_P2.54mm_Horizontal
Connections:
- removed net VS: J10.1 (Pin_1), J10.2 (Pin_2), J3.1 (Pin_1), J4.1 (Pin_1), J5.1 (Pin_1), J6.1 (Pin_1), J7.1 (Pin_1), J8.1 (Pin_1), J9.1 (Pin_1), J9.2 (Pin_2)
- new net VS1: J3.1 (Pin_1), J6.1 (Pin_1), J9.1 (Pin_1)
- new net VS2: J10.2 (Pin_2), J4.1 (Pin_1), J7.1 (Pin_1), J9.2 (Pin_2)
- new net VS3: J10.1 (Pin_1), J5.1 (Pin_1), J8.1 (Pin_1)

Commit message: Convert to KiCAD v9 and basic sort out of components
Parts:
- renumbered J1 to J11, R5 to R28, R6 to R29
Changed lines of the file:
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@@
 (kicad_sch
-	(version 20231120)
+	(version 20250114)
 	(generator "eeschema")
-	(generator_version "8.0")
+	(generator_version "9.0")
 	(paper "A4")
 	(junction
@@
 	(label "DIN_5V"
 		(at 38.1 149.86 0)
-		(fields_autoplaced yes)
 		(effects
 			(font
@@
 	(label "D-"
 		(at 55.88 102.87 0)
-		(fields_autoplaced yes)
 		(effects
 			(font
@@
 	(label "CLK"
 		(at 93.98 165.1 0)
-		(fields_autoplaced yes)
 		(effects
 			(font
@@
 	(label "DOUT"
 		(at 93.98 160.02 0)
-		(fields_autoplaced yes)
 		(effects
 			(font
@@
 	(label "VS3"
 		(at 224.79 119.38 0)
-		(fields_autoplaced yes)
 		(effects
 			(font
@@
 	(label "CLK_5V"
 		(at 38.1 177.8 0)
-		(fields_autoplaced yes)
 		(effects
 			(font
@@
 	(label "DIN_5V"
 		(at 66.04 154.94 180)
-		(fields_autoplaced yes)
 		(effects
 			(font
@@
 	(label "DOUT_5V"
 		(at 66.04 160.02 180)
-		(fields_autoplaced yes)
 		(effects
 			(font
@@
 	(label "VS2"
 		(at 224.79 72.39 0)
-		(fields_autoplaced yes)
 		(effects
 			(font
@@
 	(label "VS3"
 		(at 60.96 62.23 0)
-		(fields_autoplaced yes)
 		(effects
 			(font
@@
 	(label "CLK_5V"
 		(at 66.04 165.1 180)
-		(fields_autoplaced yes)
 		(effects
 			(font
@@
 	(label "D-"
 		(at 105.41 83.82 180)
-		(fields_autoplaced yes)
 		(effects
 			(font
@@
 	(label "VS1"
 		(at 224.79 26.67 0)
-		(fields_autoplaced yes)
 		(effects
 			(font
@@
 	(label "DOUT_5V"
 		(at 38.1 175.26 0)
-		(fields_autoplaced yes)
 		(effects
 			(font
@@
 	(label "DIN"
 		(at 93.98 154.94 0)
-		(fields_autoplaced yes)
 		(effects
 			(font
@@
 	(label "CLK"
 		(at 104.14 113.03 180)
-		(fields_autoplaced yes)
 		(effects
 			(font
@@
 	(label "VS1"
 		(at 60.96 21.59 0)
-		(fields_autoplaced yes)
 		(effects
 			(font
@@
 	(label "D+"
 		(at 55.88 105.41 0)
-		(fields_autoplaced yes)
 		(effects
 			(font
@@
 	(label "VS3"
 		(at 45.72 39.37 0)
-		(fields_autoplaced yes)
 		(effects
 			(font
@@
 	(label "VS2"
 		(at 60.96 41.91 0)
-		(fields_autoplaced yes)
 		(effects
 			(font
@@
 	(label "CLK_5V"
 		(at 38.1 152.4 0)
-		(fields_autoplaced yes)
 		(effects
 			(font
@@
 	(label "VS2"
 		(at 35.56 39.37 0)
-		(fields_autoplaced yes)
 		(effects
 			(font
@@
 	(label "VS1"
 		(at 25.4 39.37 0)
-		(fields_autoplaced yes)
 		(effects
 			(font
@@
 	(label "DOUT"
 		(at 104.14 118.11 180)
-		(fields_autoplaced yes)
 		(effects
 			(font
@@
 	(label "DIN"
 		(at 104.14 115.57 180)
-		(fields_autoplaced yes)
 		(effects
 			(font
@@
 	(label "D+"
 		(at 105.41 81.28 180)
-		(fields_autoplaced yes)
 		(effects
 			(font
@@
 		(on_board yes)
 		(dnp no)
-		(property "Reference" "#PWR0116"
+		(property "Reference" "#PWR073"
 			(at 38.1 134.62 0)
 			(effects
@@
 		(on_board yes)
 		(dnp no)
-		(property "Reference" "R6"
+		(property "Reference" "R29"
 			(at 76.708 100.4316 0)
 			(effects
@@
 		(on_board yes)
 		(dnp no)
-		(property "Reference" "J1"
+		(property "Reference" "J11"
 			(at 40.8178 80.8482 0)
 			(effects
@@
 		(on_board yes)
 		(dnp no)
-		(property "Reference" "R5"
+		(property "Reference" "R28"
 			(at 67.818 100.4316 0)
 			(effects
@@
 		(on_board yes)
 		(dnp no)
-		(property "Reference" "#PWR0117"
+		(property "Reference" "#PWR074"
 			(at 55.88 91.44 0)
 			(effects
@@
 		(on_board yes)
 		(dnp no)
-		(property "Reference" "#PWR02"
+		(property "Reference" "#PWR075"
 			(at 66.04 114.3 0)
 			(effects
@@
 		(on_board yes)
 		(dnp no)
-		(property "Reference" "#PWR0118"
+		(property "Reference" "#PWR076"
 			(at 74.93 114.3 0)
 			(effects
@@
 		(at 185.42 124.46)
 		(size 35.56 17.78)
+		(exclude_from_sim no)
+		(in_bom yes)
+		(on_board yes)
+		(dnp no)
 		(fields_autoplaced yes)
 		(stroke
@@
 		(at 109.22 53.34)
 		(size 50.8 92.71)
+		(exclude_from_sim no)
+		(in_bom yes)
+		(on_board yes)
+		(dnp no)
 		(fields_autoplaced yes)
 		(stroke
@@
 		(at 185.42 77.47)
 		(size 35.56 17.78)
+		(exclude_from_sim no)
+		(in_bom yes)
+		(on_board yes)
+		(dnp no)
 		(fields_autoplaced yes)
 		(stroke
@@
 		(at 185.42 31.75)
 		(size 35.56 17.78)
+		(exclude_from_sim no)
+		(in_bom yes)
+		(on_board yes)
+		(dnp no)
 		(fields_autoplaced yes)
 		(stroke
@@
 		)
 	)
+	(embedded_fonts no)
 )

Commit message: Additional layout
Parts:
- R28, R29: footprint Resistor_SMD:R_0805_2012Metric -> Resistor_SMD:R_0603_1608Metric
Changed lines of the file:
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@@
 			)
 		)
-		(property "Footprint" "Resistor_SMD:R_0805_2012Metric"
+		(property "Footprint" "Resistor_SMD:R_0603_1608Metric"
 			(at 73.152 101.6 90)
 			(effects
@@
 			)
 		)
-		(property "Footprint" "Resistor_SMD:R_0805_2012Metric"
+		(property "Footprint" "Resistor_SMD:R_0603_1608Metric"
 			(at 64.262 101.6 90)
 			(effects
