File: SmartishFairy.kicad_sch (KiCad schematic)
At the start: 15 parts, among them J10 Conn_01x02_Pin, J11 USB_C_Receptacle_USB2.0, J13 Data_In, J14 Data_Out, J15 Ctl_Pwr, J3 IN1, J4 IN2, J5 IN3, J6 OUT1, J7 OUT2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

Commit message: Added a few JLC part number
Parts:
- R28, R29: LCSC C139928 -> (none)
Changed lines of the file:
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@@
 			)
 		)
-		(property "LCSC" "C139928"
+		(property "LCSC" ""
 			(at 74.93 101.6 0)
 			(effects
@@
 			)
 		)
-		(property "LCSC" "C139928"
+		(property "LCSC" ""
 			(at 66.04 101.6 0)
 			(effects

Commit message: More updates
Placed more components
Updated 3D models
Parts:
- added H1, H2, H3, H4: MountingHole, MountingHole:MountingHole_3mm, symbol Mechanical:MountingHole
- R28, R29: footprint Resistor_SMD:R_0603_1608Metric -> Resistor_SMD:R_0402_1005Metric
