File: driver.kicad_sch (KiCad schematic)
At the start: 14 parts, among them U2 L6226Q

Commit message: ECR fixes
Parts:
- C1, C2, C3, C4, C5, C6: footprint (none) -> Capacitor_SMD:C_0805_2012Metric
- R1, R2, R3, R4, R5, R6: footprint (none) -> Resistor_SMD:R_0805_2012Metric
Changed lines of the file:
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@@
       (effects (font (size 1.27 1.27)) (justify left))
     )
-    (property "Footprint" "" (at 121.6152 123.19 0)
+    (property "Footprint" "Capacitor_SMD:C_0805_2012Metric" (at 121.6152 123.19 0)
       (effects (font (size 1.27 1.27)) hide)
     )
@@
       (effects (font (size 1.27 1.27)) (justify right))
     )
-    (property "Footprint" "" (at 114.6048 49.53 0)
+    (property "Footprint" "Capacitor_SMD:C_0805_2012Metric" (at 114.6048 49.53 0)
       (effects (font (size 1.27 1.27)) hide)
     )
@@
       (effects (font (size 1.27 1.27)) (justify left))
     )
-    (property "Footprint" "" (at 103.378 118.11 90)
+    (property "Footprint" "Resistor_SMD:R_0805_2012Metric" (at 103.378 118.11 90)
       (effects (font (size 1.27 1.27)) hide)
     )
@@
       (effects (font (size 1.27 1.27)) (justify left))
     )
-    (property "Footprint" "" (at 168.6052 58.42 0)
+    (property "Footprint" "Capacitor_SMD:C_0805_2012Metric" (at 168.6052 58.42 0)
       (effects (font (size 1.27 1.27)) hide)
     )
@@
       (effects (font (size 1.27 1.27)))
     )
-    (property "Footprint" "" (at 106.68 97.282 90)
+    (property "Footprint" "Resistor_SMD:R_0805_2012Metric" (at 106.68 97.282 90)
       (effects (font (size 1.27 1.27)) hide)
     )
@@
       (effects (font (size 1.27 1.27)) (justify right))
     )
-    (property "Footprint" "" (at 138.938 119.38 90)
+    (property "Footprint" "Resistor_SMD:R_0805_2012Metric" (at 138.938 119.38 90)
       (effects (font (size 1.27 1.27)) hide)
     )
@@
       (effects (font (size 1.27 1.27)))
     )
-    (property "Footprint" "" (at 143.51 57.4548 0)
+    (property "Footprint" "Capacitor_SMD:C_0805_2012Metric" (at 143.51 57.4548 0)
       (effects (font (size 1.27 1.27)) hide)
     )
@@
       (effects (font (size 1.27 1.27)) (justify left))
     )
-    (property "Footprint" "" (at 94.488 118.11 90)
+    (property "Footprint" "Resistor_SMD:R_0805_2012Metric" (at 94.488 118.11 90)
       (effects (font (size 1.27 1.27)) hide)
     )
@@
       (effects (font (size 1.27 1.27)))
     )
-    (property "Footprint" "" (at 106.68 84.582 90)
+    (property "Footprint" "Resistor_SMD:R_0805_2012Metric" (at 106.68 84.582 90)
       (effects (font (size 1.27 1.27)) hide)
     )
@@
       (effects (font (size 1.27 1.27)) (justify right))
     )
-    (property "Footprint" "" (at 131.318 119.38 90)
+    (property "Footprint" "Resistor_SMD:R_0805_2012Metric" (at 131.318 119.38 90)
       (effects (font (size 1.27 1.27)) hide)
     )
@@
       (effects (font (size 1.27 1.27)))
     )
-    (property "Footprint" "" (at 171.45 33.3248 0)
+    (property "Footprint" "Capacitor_SMD:C_0805_2012Metric" (at 171.45 33.3248 0)
       (effects (font (size 1.27 1.27)) hide)
     )
@@
       (effects (font (size 1.27 1.27)) (justify left))
     )
-    (property "Footprint" "" (at 112.7252 123.19 0)
-      (effects (font (size 1.27 1.27)) hide)
-    )
+    (property "Footprint" "Capacitor_SMD:C_0805_2012Metric" (at 112.7252 123.19 0)
+      (effects (font (size 1.27 1.27)) hide)
+    )

Commit message: Layout WIP
Parts:
- C14: renamed from C4; footprint Capacitor_SMD:C_0805_2012Metric -> Capacitor_SMD:CP_Elec_5x4.4
- renumbered C2 to C13, C1 to C15, C6 to C16, C5 to C17, C3 to C18, D1 to D3, R5 to R13, R4 to R14, R1 to R15, R6 to R16, R3 to R17, R2 to R18, U2 to U7

Commit message: Convert to KiCAD v9 and basic sort out of components
Parts:
- renumbered C15 to C1, C13 to C2, C18 to C3, C14 to C4, C17 to C5, C16 to C6, D3 to D1, R15 to R1, R18 to R2, R17 to R3, R14 to R4, R13 to R5, R16 to R6, U7 to U5

Commit message: Additional layout
Parts:
- C1, C2, C3, C5, C6: footprint Capacitor_SMD:C_0805_2012Metric -> Capacitor_SMD:C_0603_1608Metric
- R1, R2, R3, R4, R5, R6: footprint Resistor_SMD:R_0805_2012Metric -> Resistor_SMD:R_0603_1608Metric
Changed lines of the file:
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@@
 			)
 		)
-		(property "Footprint" "Capacitor_SMD:C_0805_2012Metric"
+		(property "Footprint" "Capacitor_SMD:C_0603_1608Metric"
 			(at 121.6152 123.19 0)
 			(effects
@@
 			)
 		)
-		(property "Footprint" "Resistor_SMD:R_0805_2012Metric"
+		(property "Footprint" "Resistor_SMD:R_0603_1608Metric"
 			(at 103.378 118.11 90)
 			(effects
@@
 			)
 		)
-		(property "Footprint" "Capacitor_SMD:C_0805_2012Metric"
+		(property "Footprint" "Capacitor_SMD:C_0603_1608Metric"
 			(at 168.6052 58.42 0)
 			(effects
@@
 			)
 		)
-		(property "Footprint" "Resistor_SMD:R_0805_2012Metric"
+		(property "Footprint" "Resistor_SMD:R_0603_1608Metric"
 			(at 106.68 97.282 90)
 			(effects
@@
 			)
 		)
-		(property "Footprint" "Resistor_SMD:R_0805_2012Metric"
+		(property "Footprint" "Resistor_SMD:R_0603_1608Metric"
 			(at 138.938 119.38 90)
 			(effects
@@
 			)
 		)
-		(property "Footprint" "Capacitor_SMD:C_0805_2012Metric"
+		(property "Footprint" "Capacitor_SMD:C_0603_1608Metric"
 			(at 143.51 57.4548 0)
 			(effects
@@
 			)
 		)
-		(property "Footprint" "Resistor_SMD:R_0805_2012Metric"
+		(property "Footprint" "Resistor_SMD:R_0603_1608Metric"
 			(at 94.488 118.11 90)
 			(effects
@@
 			)
 		)
-		(property "Footprint" "Resistor_SMD:R_0805_2012Metric"
+		(property "Footprint" "Resistor_SMD:R_0603_1608Metric"
 			(at 106.68 84.582 90)
 			(effects
@@
 			)
 		)
-		(property "Footprint" "Resistor_SMD:R_0805_2012Metric"
+		(property "Footprint" "Resistor_SMD:R_0603_1608Metric"
 			(at 131.318 119.38 90)
 			(effects
@@
 			)
 		)
-		(property "Footprint" "Capacitor_SMD:C_0805_2012Metric"
+		(property "Footprint" "Capacitor_SMD:C_0603_1608Metric"
 			(at 171.45 33.3248 0)
 			(effects
@@
 			)
 		)
-		(property "Footprint" "Capacitor_SMD:C_0805_2012Metric"
+		(property "Footprint" "Capacitor_SMD:C_0603_1608Metric"
 			(at 112.7252 123.19 0)
 			(effects
